Commit message: some manual edits on urdf output ver0.

File: assembly_models/picknplace/bricks/urdf/brick_demo.urdf (robot description, URDF)
Before this commit: robot brick_demo, 39 links, 38 joints
Links:
- removed link ws_place_support_object_0
- removed link ws_place_support_object_1
- removed link ws_place_support_object_10
- removed link ws_place_support_object_11
- removed link ws_place_support_object_2
- removed link ws_place_support_object_3
- removed link ws_place_support_object_4
- removed link ws_place_support_object_5
- removed link ws_place_support_object_6
- removed link ws_place_support_object_7
- removed link ws_place_support_object_8
- removed link ws_place_support_object_9
- link ws_pick_element_0: geometry collision mesh filename=/home/yijiangh/catkin_ws/src/assembly-instances/assembly_mo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 scale=0.001 0.001 0.001; visual mesh filename=/home/yijiangh/catkin_ws/src/assembly-instances/assembly_mo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 scale=0.001 0.001 0.001
- link ws_pick_element_1: geometry collision mesh filename=/home/yijiangh/catkin_ws/src/assembly-instances/assembly_mo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 scale=0.001 0.001 0.001; visual mesh filename=/home/yijiangh/catkin_ws/src/assembly-instances/assembly_mo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 scale=0.001 0.001 0.001
- link ws_pick_element_10: geometry collision mesh filename=/home/yijiangh/catkin_ws/src/assembly-instances/assembly_mo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 scale=0.001 0.001 0.001; visual mesh filename=/home/yijiangh/catkin_ws/src/assembly-instances/assembly_mo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 scale=0.001 0.001 0.001
- link ws_pick_element_11: geometry collision mesh filename=/home/yijiangh/catkin_ws/src/assembly-instances/assembly_mo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 scale=0.001 0.001 0.001; visual mesh filename=/home/yijiangh/catkin_ws/src/assembly-instances/assembly_mo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 scale=0.001 0.001 0.001
- link ws_pick_element_2: geometry collision mesh filename=/home/yijiangh/catkin_ws/src/assembly-instances/assembly_mo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 scale=0.001 0.001 0.001; visual mesh filename=/home/yijiangh/catkin_ws/src/assembly-instances/assembly_mo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 scale=0.001 0.001 0.001
- link ws_pick_element_3: geometry collision mesh filename=/home/yijiangh/catkin_ws/src/assembly-instances/assembly_mo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 scale=0.001 0.001 0.001; visual mesh filename=/home/yijiangh/catkin_ws/src/assembly-instances/assembly_mo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 scale=0.001 0.001 0.001
- link ws_pick_element_4: geometry collision mesh filename=/home/yijiangh/catkin_ws/src/assembly-instances/assembly_mo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 scale=0.001 0.001 0.001; visual mesh filename=/home/yijiangh/catkin_ws/src/assembly-instances/assembly_mo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 scale=0.001 0.001 0.001
- link ws_pick_element_5: geometry collision mesh filename=/home/yijiangh/catkin_ws/src/assembly-instances/assembly_mo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 scale=0.001 0.001 0.001; visual mesh filename=/home/yijiangh/catkin_ws/src/assembly-instances/assembly_mo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 scale=0.001 0.001 0.001
- link ws_pick_element_6: geometry collision mesh filename=/home/yijiangh/catkin_ws/src/assembly-instances/assembly_mo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 scale=0.001 0.001 0.001; visual mesh filename=/home/yijiangh/catkin_ws/src/assembly-instances/assembly_mo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 scale=0.001 0.001 0.001
- link ws_pick_element_7: geometry collision mesh filename=/home/yijiangh/catkin_ws/src/assembly-instances/assembly_mo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 scale=0.001 0.001 0.001; visual mesh filename=/home/yijiangh/catkin_ws/src/assembly-instances/assembly_mo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 scale=0.001 0.001 0.001
- link ws_pick_element_8: geometry collision mesh filename=/home/yijiangh/catkin_ws/src/assembly-instances/assembly_mo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 scale=0.001 0.001 0.001; visual mesh filename=/home/yijiangh/catkin_ws/src/assembly-instances/assembly_mo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 scale=0.001 0.001 0.001
- link ws_pick_element_9: geometry collision mesh filename=/home/yijiangh/catkin_ws/src/assembly-instances/assembly_mo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 scale=0.001 0.001 0.001; visual mesh filename=/home/yijiangh/catkin_ws/src/assembly-instances/assembly_mo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 scale=0.001 0.001 0.001
- link ws_pick_support_object_0: geometry collision mesh filename=/home/yijiangh/catkin_ws/src/assembly-instances/assembly_mo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 scale=0.001 0.001 0.001; visual mesh filename=/home/yijiangh/catkin_ws/src/assembly-instances/assembly_mo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 scale=0.001 0.001 0.001
- link ws_place_element_0: geometry collision mesh filename=/home/yijiangh/catkin_ws/src/assembly-instances/assembly_mo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 scale=0.001 0.001 0.001; visual mesh filename=/home/yijiangh/catkin_ws/src/assembly-instances/assembly_mo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 scale=0.001 0.001 0.001
- link ws_place_element_1: geometry collision mesh filename=/home/yijiangh/catkin_ws/src/assembly-instances/assembly_mo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 scale=0.001 0.001 0.001; visual mesh filename=/home/yijiangh/catkin_ws/src/assembly-instances/assembly_mo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 scale=0.001 0.001 0.001
- link ws_place_element_10: geometry collision mesh filename=/home/yijiangh/catkin_ws/src/assembly-instances/assembly_mo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 scale=0.001 0.001 0.001; visual mesh filename=/home/yijiangh/catkin_ws/src/assembly-instances/assembly_mo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 scale=0.001 0.001 0.001
- link ws_place_element_11: geometry collision mesh filename=/home/yijiangh/catkin_ws/src/assembly-instances/assembly_mo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 scale=0.001 0.001 0.001; visual mesh filename=/home/yijiangh/catkin_ws/src/assembly-instances/assembly_mo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 scale=0.001 0.001 0.001
- link ws_place_element_2: geometry collision mesh filename=/home/yijiangh/catkin_ws/src/assembly-instances/assembly_mo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 scale=0.001 0.001 0.001; visual mesh filename=/home/yijiangh/catkin_ws/src/assembly-instances/assembly_mo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 scale=0.001 0.001 0.001
- link ws_place_element_3: geometry collision mesh filename=/home/yijiangh/catkin_ws/src/assembly-instances/assembly_mo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 scale=0.001 0.001 0.001; visual mesh filename=/home/yijiangh/catkin_ws/src/assembly-instances/assembly_mo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 scale=0.001 0.001 0.001
- link ws_place_element_4: geometry collision mesh filename=/home/yijiangh/catkin_ws/src/assembly-instances/assembly_mo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 scale=0.001 0.001 0.001; visual mesh filename=/home/yijiangh/catkin_ws/src/assembly-instances/assembly_mo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 scale=0.001 0.001 0.001
- link ws_place_element_5: geometry collision mesh filename=/home/yijiangh/catkin_ws/src/assembly-instances/assembly_mo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 scale=0.001 0.001 0.001; visual mesh filename=/home/yijiangh/catkin_ws/src/assembly-instances/assembly_mo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 scale=0.001 0.001 0.001
- link ws_place_element_6: geometry collision mesh filename=/home/yijiangh/catkin_ws/src/assembly-instances/assembly_mo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 scale=0.001 0.001 0.001; visual mesh filename=/home/yijiangh/catkin_ws/src/assembly-instances/assembly_mo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 scale=0.001 0.001 0.001
- link ws_place_element_7: geometry collision mesh filename=/home/yijiangh/catkin_ws/src/assembly-instances/assembly_mo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 scale=0.001 0.001 0.001; visual mesh filename=/home/yijiangh/catkin_ws/src/assembly-instances/assembly_mo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 scale=0.001 0.001 0.001
- link ws_place_element_8: geometry collision mesh filename=/home/yijiangh/catkin_ws/src/assembly-instances/assembly_mo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 scale=0.001 0.001 0.001; visual mesh filename=/home/yijiangh/catkin_ws/src/assembly-instances/assembly_mo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 scale=0.001 0.001 0.001
- link ws_place_element_9: geometry collision mesh filename=/home/yijiangh/catkin_ws/src/assembly-instances/assembly_mo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 scale=0.001 0.001 0.001; visual mesh filename=/home/yijiangh/catkin_ws/src/assembly-instances/assembly_mo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 scale=0.001 0.001 0.001
Joints:
- removed joint ws_base2place_support_object_0
- removed joint ws_base2place_support_object_1
- removed joint ws_base2place_support_object_10
- removed joint ws_base2place_support_object_11
- removed joint ws_base2place_support_object_2
- removed joint ws_base2place_support_object_3
- removed joint ws_base2place_support_object_4
- removed joint ws_base2place_support_object_5
- removed joint ws_base2place_support_object_6
- removed joint ws_base2place_support_object_7
- removed joint ws_base2place_support_object_8
- removed joint ws_base2place_support_object_9

File: assembly_models/picknplace/bricks/urdf/brick_demo.xacro (robot description, xacro)
@@ -1,3 +1,3 @@
-﻿<?xml version="1.0" encoding="utf-8"?>
+﻿<?xml version="1.0" ?>
 <robot name="brick_demo" xmlns:xacro="http://wiki.ros.org/xacro">
 	<xacro:include filename="$(find assembly-instances)/assembly_models/picknplace/bricks/urdf/brick_demo_geometry.xacro" />

File: assembly_models/picknplace/bricks/urdf/brick_demo_geometry.xacro (robot description, xacro)
@@ -1,3 +1,3 @@
-﻿<?xml version="1.0" encoding="utf-8"?>
+﻿<?xml version="1.0" ?>
 <robot xmlns:xacro="http://wiki.ros.org/xacro">
 	<xacro:macro name="brick_demo_geometry" params="prefix">
@@ -428,208 +428,4 @@
 			<origin xyz="0 0 0" rpy="0 0 0" />
 		</joint>
-		<link name="${prefix}place_support_object_0">
-			<visual>
-				<geometry>
-					<mesh filename="$(find assembly-instances)/assembly_models/picknplace/bricks/meshes/collision/pick_left_over_bricks_0.stl" scale="0.001 0.001 0.001" />
-				</geometry>
-			</visual>
-			<collision>
-				<geometry>
-					<mesh filename="$(find assembly-instances)/assembly_models/picknplace/bricks/meshes/collision/pick_left_over_bricks_0.stl" scale="0.001 0.001 0.001" />
-				</geometry>
-			</collision>
-		</link>
-		<joint name="${prefix}base2place_support_object_0" type="fixed">
-			<parent link="${prefix}base_link" />
-			<child link="${prefix}place_support_object_0" />
-			<origin xyz="0 0 0" rpy="0 0 0" />
-		</joint>
-		<link name="${prefix}place_support_object_1">
-			<visual>
-				<geometry>
-					<mesh filename="$(find assembly-instances)/assembly_models/picknplace/bricks/meshes/collision/pick_left_over_bricks_1.stl" scale="0.001 0.001 0.001" />
-				</geometry>
-			</visual>
-			<collision>
-				<geometry>
-					<mesh filename="$(find assembly-instances)/assembly_models/picknplace/bricks/meshes/collision/pick_left_over_bricks_1.stl" scale="0.001 0.001 0.001" />
-				</geometry>
-			</collision>
-		</link>
-		<joint name="${prefix}base2place_support_object_1" type="fixed">
-			<parent link="${prefix}base_link" />
-			<child link="${prefix}place_support_object_1" />
-			<origin xyz="0 0 0" rpy="0 0 0" />
-		</joint>
-		<link name="${prefix}place_support_object_2">
-			<visual>
-				<geometry>
-					<mesh filename="$(find assembly-instances)/assembly_models/picknplace/bricks/meshes/collision/pick_left_over_bricks_4.stl" scale="0.001 0.001 0.001" />
-				</geometry>
-			</visual>
-			<collision>
-				<geometry>
-					<mesh filename="$(find assembly-instances)/assembly_models/picknplace/bricks/meshes/collision/pick_left_over_bricks_4.stl" scale="0.001 0.001 0.001" />
-				</geometry>
-			</collision>
-		</link>
-		<joint name="${prefix}base2place_support_object_2" type="fixed">
-			<parent link="${prefix}base_link" />
-			<child link="${prefix}place_support_object_2" />
-			<origin xyz="0 0 0" rpy="0 0 0" />
-		</joint>
-		<link name="${prefix}place_support_object_3">
-			<visual>
-				<geometry>
-					<mesh filename="$(find assembly-instances)/assembly_models/picknplace/bricks/meshes/collision/pick_left_over_bricks_2.stl" scale="0.001 0.001 0.001" />
-				</geometry>
-			</visual>
-			<collision>
-				<geometry>
-					<mesh filename="$(find assembly-instances)/assembly_models/picknplace/bricks/meshes/collision/pick_left_over_bricks_2.stl" scale="0.001 0.001 0.001" />
-				</geometry>
-			</collision>
-		</link>
-		<joint name="${prefix}base2place_support_object_3" type="fixed">
-			<parent link="${prefix}base_link" />
-			<child link="${prefix}place_support_object_3" />
-			<origin xyz="0 0 0" rpy="0 0 0" />
-		</joint>
-		<link name="${prefix}place_support_object_4">
-			<visual>
-				<geometry>
-					<mesh filename="$(find assembly-instances)/assembly_models/picknplace/bricks/meshes/collision/pick_left_over_bricks_5.stl" scale="0.001 0.001 0.001" />
-				</geometry>
-			</visual>
-			<collision>
-				<geometry>
-					<mesh filename="$(find assembly-instances)/assembly_models/picknplace/bricks/meshes/collision/pick_left_over_bricks_5.stl" scale="0.001 0.001 0.001" />
-				</geometry>
-			</collision>
-		</link>
-		<joint name="${prefix}base2place_support_object_4" type="fixed">
-			<parent link="${prefix}base_link" />
-			<child link="${prefix}place_support_object_4" />
-			<origin xyz="0 0 0" rpy="0 0 0" />
-		</joint>
-		<link name="${prefix}place_support_object_5">
-			<visual>
-				<geometry>
-					<mesh filename="$(find assembly-instances)/assembly_models/picknplace/bricks/meshes/collision/pick_left_over_bricks_3.stl" scale="0.001 0.001 0.001" />
-				</geometry>
-			</visual>
-			<collision>
-				<geometry>
-					<mesh filename="$(find assembly-instances)/assembly_models/picknplace/bricks/meshes/collision/pick_left_over_bricks_3.stl" scale="0.001 0.001 0.001" />
-				</geometry>
-			</collision>
-		</link>
-		<joint name="${prefix}base2place_support_object_5" type="fixed">
-			<parent link="${prefix}base_link" />
-			<child link="${prefix}place_support_object_5" />
-			<origin xyz="0 0 0" rpy="0 0 0" />
-		</joint>
-		<link name="${prefix}place_support_object_6">
-			<visual>
-				<geometry>
-					<mesh filename="$(find assembly-instances)/assembly_models/picknplace/bricks/meshes/collision/pick_left_over_bricks_6.stl" scale="0.001 0.001 0.001" />
-				</geometry>
-			</visual>
-			<collision>
-				<geometry>
-					<mesh filename="$(find assembly-instances)/assembly_models/picknplace/bricks/meshes/collision/pick_left_over_bricks_6.stl" scale="0.001 0.001 0.001" />
-				</geometry>
-			</collision>
-		</link>
-		<joint name="${prefix}base2place_support_object_6" type="fixed">
-			<parent link="${prefix}base_link" />
-			<child link="${prefix}place_support_object_6" />
-			<origin xyz="0 0 0" rpy="0 0 0" />
-		</joint>
-		<link name="${prefix}place_support_object_7">
-			<visual>
-				<geometry>
-					<mesh filename="$(find assembly-instances)/assembly_models/picknplace/bricks/meshes/collision/pick_left_over_bricks_7.stl" scale="0.001 0.001 0.001" />
-				</geometry>
-			</visual>
-			<collision>
-				<geometry>
-					<mesh filename="$(find assembly-instances)/assembly_models/picknplace/bricks/meshes/collision/pick_left_over_bricks_7.stl" scale="0.001 0.001 0.001" />
-				</geometry>
-			</collision>
-		</link>
-		<joint name="${prefix}base2place_support_object_7" type="fixed">
-			<parent link="${prefix}base_link" />
-			<child link="${prefix}place_support_object_7" />
-			<origin xyz="0 0 0" rpy="0 0 0" />
-		</joint>
-		<link name="${prefix}place_support_object_8">
-			<visual>
-				<geometry>
-					<mesh filename="$(find assembly-instances)/assembly_models/picknplace/bricks/meshes/collision/pick_left_over_bricks_8.stl" scale="0.001 0.001 0.001" />
-				</geometry>
-			</visual>
-			<collision>
-				<geometry>
-					<mesh filename="$(find assembly-instances)/assembly_models/picknplace/bricks/meshes/collision/pick_left_over_bricks_8.stl" scale="0.001 0.001 0.001" />
-				</geometry>
-			</collision>
-		</link>
-		<joint name="${prefix}base2place_support_object_8" type="fixed">
-			<parent link="${prefix}base_link" />
-			<child link="${prefix}place_support_object_8" />
-			<origin xyz="0 0 0" rpy="0 0 0" />
-		</joint>
-		<link name="${prefix}place_support_object_9">
-			<visual>
-				<geometry>
-					<mesh filename="$(find assembly-instances)/assembly_models/picknplace/bricks/meshes/collision/pick_left_over_bricks_9.stl" scale="0.001 0.001 0.001" />
-				</geometry>
-			</visual>
-			<collision>
-				<geometry>
-					<mesh filename="$(find assembly-instances)/assembly_models/picknplace/bricks/meshes/collision/pick_left_over_bricks_9.stl" scale="0.001 0.001 0.001" />
-				</geometry>
-			</collision>
-		</link>
-		<joint name="${prefix}base2place_support_object_9" type="fixed">
-			<parent link="${prefix}base_link" />
-			<child link="${prefix}place_support_object_9" />
-			<origin xyz="0 0 0" rpy="0 0 0" />
-		</joint>
-		<link name="${prefix}place_support_object_10">
-			<visual>
-				<geometry>
-					<mesh filename="$(find assembly-instances)/assembly_models/picknplace/bricks/meshes/collision/pick_left_over_bricks_10.stl" scale="0.001 0.001 0.001" />
-				</geometry>
-			</visual>
-			<collision>
-				<geometry>
-					<mesh filename="$(find assembly-instances)/assembly_models/picknplace/bricks/meshes/collision/pick_left_over_bricks_10.stl" scale="0.001 0.001 0.001" />
-				</geometry>
-			</collision>
-		</link>
-		<joint name="${prefix}base2place_support_object_10" type="fixed">
-			<parent link="${prefix}base_link" />
-			<child link="${prefix}place_support_object_10" />
-			<origin xyz="0 0 0" rpy="0 0 0" />
-		</joint>
-		<link name="${prefix}place_support_object_11">
-			<visual>
-				<geometry>
-					<mesh filename="$(find assembly-instances)/assembly_models/picknplace/bricks/meshes/collision/pick_left_over_bricks_11.stl" scale="0.001 0.001 0.001" />
-				</geometry>
-			</visual>
-			<collision>
-				<geometry>
-					<mesh filename="$(find assembly-instances)/assembly_models/picknplace/bricks/meshes/collision/pick_left_over_bricks_11.stl" scale="0.001 0.001 0.001" />
-				</geometry>
-			</collision>
-		</link>
-		<joint name="${prefix}base2place_support_object_11" type="fixed">
-			<parent link="${prefix}base_link" />
-			<child link="${prefix}place_support_object_11" />
-			<origin xyz="0 0 0" rpy="0 0 0" />
-		</joint>
 	</xacro:macro>
 </robot>
