Commit message: made into a ros package.

File: assembly_models/picknplace/bricks/urdf/brick_demo.xacro (robot description, xacro)
@@ -1,779 +1,11 @@
 ﻿<?xml version="1.0" encoding="utf-8"?>
-<robot xmlns:xacro="http://wiki.ros.org/xacro">
-	<xacro:macro name="brick_demo" params="prefix">
-		<link name="${prefix}base_link" />
-		<link name="${prefix}pick_element_0">
-			<visual>
-				<geometry>
-					<mesh filename="package://assembly-instances/assembly_models/picknplace/bricks/meshes/collision/element_pick_0.stl" scale="0.001 0.001 0.001" />
-				</geometry>
-			</visual>
-			<collision>
-				<geometry>
-					<mesh filename="package://assembly-instances/assembly_models/picknplace/bricks/meshes/collision/element_pick_0.stl" scale="0.001 0.001 0.001" />
-				</geometry>
-			</collision>
-		</link>
-		<joint name="${prefix}base2pick_element_0">
-			<parent link="${prefix}base_link" />
-			<child link="${prefix}pick_element_0" />
-			<origin xyz="0 0 0" rpy="0 0 0" />
-		</joint>
-		<link name="${prefix}place_element_0">
-			<visual>
-				<geometry>
-					<mesh filename="package://assembly-instances/assembly_models/picknplace/bricks/meshes/collision/element_place_0.stl" scale="0.001 0.001 0.001" />
-				</geometry>
-			</visual>
-			<collision>
-				<geometry>
-					<mesh filename="package://assembly-instances/assembly_models/picknplace/bricks/meshes/collision/element_place_0.stl" scale="0.001 0.001 0.001" />
-				</geometry>
-			</collision>
-		</link>
-		<link name="${prefix}place_element_0">
-			<visual>
-				<geometry>
-					<mesh filename="package://assembly-instances/assembly_models/picknplace/bricks/meshes/collision/element_place_0.stl" scale="0.001 0.001 0.001" />
-				</geometry>
-			</visual>
-			<collision>
-				<geometry>
-					<mesh filename="package://assembly-instances/assembly_models/picknplace/bricks/meshes/collision/element_place_0.stl" scale="0.001 0.001 0.001" />
-				</geometry>
-			</collision>
-		</link>
-		<joint name="${prefix}base2place_element_0">
-			<parent link="${prefix}base_link" />
-			<child link="${prefix}place_element_0" />
-			<origin xyz="0 0 0" rpy="0 0 0" />
-		</joint>
-		<link name="${prefix}pick_element_1">
-			<visual>
-				<geometry>
-					<mesh filename="package://assembly-instances/assembly_models/picknplace/bricks/meshes/collision/element_pick_1.stl" scale="0.001 0.001 0.001" />
-				</geometry>
-			</visual>
-			<collision>
-				<geometry>
-					<mesh filename="package://assembly-instances/assembly_models/picknplace/bricks/meshes/collision/element_pick_1.stl" scale="0.001 0.001 0.001" />
-				</geometry>
-			</collision>
-		</link>
-		<joint name="${prefix}base2pick_element_1">
-			<parent link="${prefix}base_link" />
-			<child link="${prefix}pick_element_1" />
-			<origin xyz="0 0 0" rpy="0 0 0" />
-		</joint>
-		<link name="${prefix}place_element_1">
-			<visual>
-				<geometry>
-					<mesh filename="package://assembly-instances/assembly_models/picknplace/bricks/meshes/collision/element_place_1.stl" scale="0.001 0.001 0.001" />
-				</geometry>
-			</visual>
-			<collision>
-				<geometry>
-					<mesh filename="package://assembly-instances/assembly_models/picknplace/bricks/meshes/collision/element_place_1.stl" scale="0.001 0.001 0.001" />
-				</geometry>
-			</collision>
-		</link>
-		<link name="${prefix}place_element_1">
-			<visual>
-				<geometry>
-					<mesh filename="package://assembly-instances/assembly_models/picknplace/bricks/meshes/collision/element_place_1.stl" scale="0.001 0.001 0.001" />
-				</geometry>
-			</visual>
-			<collision>
-				<geometry>
-					<mesh filename="package://assembly-instances/assembly_models/picknplace/bricks/meshes/collision/element_place_1.stl" scale="0.001 0.001 0.001" />
-				</geometry>
-			</collision>
-		</link>
-		<joint name="${prefix}base2place_element_1">
-			<parent link="${prefix}base_link" />
-			<child link="${prefix}place_element_1" />
-			<origin xyz="0 0 0" rpy="0 0 0" />
-		</joint>
-		<link name="${prefix}pick_element_2">
-			<visual>
-				<geometry>
-					<mesh filename="package://assembly-instances/assembly_models/picknplace/bricks/meshes/collision/element_pick_2.stl" scale="0.001 0.001 0.001" />
-				</geometry>
-			</visual>
-			<collision>
-				<geometry>
-					<mesh filename="package://assembly-instances/assembly_models/picknplace/bricks/meshes/collision/element_pick_2.stl" scale="0.001 0.001 0.001" />
-				</geometry>
-			</collision>
-		</link>
-		<joint name="${prefix}base2pick_element_2">
-			<parent link="${prefix}base_link" />
-			<child link="${prefix}pick_element_2" />
-			<origin xyz="0 0 0" rpy="0 0 0" />
-		</joint>
-		<link name="${prefix}place_element_2">
-			<visual>
-				<geometry>
-					<mesh filename="package://assembly-instances/assembly_models/picknplace/bricks/meshes/collision/element_place_2.stl" scale="0.001 0.001 0.001" />
-				</geometry>
-			</visual>
-			<collision>
-				<geometry>
-					<mesh filename="package://assembly-instances/assembly_models/picknplace/bricks/meshes/collision/element_place_2.stl" scale="0.001 0.001 0.001" />
-				</geometry>
-			</collision>
-		</link>
-		<link name="${prefix}place_element_2">
-			<visual>
-				<geometry>
-					<mesh filename="package://assembly-instances/assembly_models/picknplace/bricks/meshes/collision/element_place_2.stl" scale="0.001 0.001 0.001" />
-				</geometry>
-			</visual>
-			<collision>
-				<geometry>
-					<mesh filename="package://assembly-instances/assembly_models/picknplace/bricks/meshes/collision/element_place_2.stl" scale="0.001 0.001 0.001" />
-				</geometry>
-			</collision>
-		</link>
-		<joint name="${prefix}base2place_element_2">
-			<parent link="${prefix}base_link" />
-			<child link="${prefix}place_element_2" />
-			<origin xyz="0 0 0" rpy="0 0 0" />
-		</joint>
-		<link name="${prefix}pick_element_3">
-			<visual>
-				<geometry>
-					<mesh filename="package://assembly-instances/assembly_models/picknplace/bricks/meshes/collision/element_pick_3.stl" scale="0.001 0.001 0.001" />
-				</geometry>
-			</visual>
-			<collision>
-				<geometry>
-					<mesh filename="package://assembly-instances/assembly_models/picknplace/bricks/meshes/collision/element_pick_3.stl" scale="0.001 0.001 0.001" />
-				</geometry>
-			</collision>
-		</link>
-		<joint name="${prefix}base2pick_element_3">
-			<parent link="${prefix}base_link" />
-			<child link="${prefix}pick_element_3" />
-			<origin xyz="0 0 0" rpy="0 0 0" />
-		</joint>
-		<link name="${prefix}place_element_3">
-			<visual>
-				<geometry>
-					<mesh filename="package://assembly-instances/assembly_models/picknplace/bricks/meshes/collision/element_place_3.stl" scale="0.001 0.001 0.001" />
-				</geometry>
-			</visual>
-			<collision>
-				<geometry>
-					<mesh filename="package://assembly-instances/assembly_models/picknplace/bricks/meshes/collision/element_place_3.stl" scale="0.001 0.001 0.001" />
-				</geometry>
-			</collision>
-		</link>
-		<link name="${prefix}place_element_3">
-			<visual>
-				<geometry>
-					<mesh filename="package://assembly-instances/assembly_models/picknplace/bricks/meshes/collision/element_place_3.stl" scale="0.001 0.001 0.001" />
-				</geometry>
-			</visual>
-			<collision>
-				<geometry>
-					<mesh filename="package://assembly-instances/assembly_models/picknplace/bricks/meshes/collision/element_place_3.stl" scale="0.001 0.001 0.001" />
-				</geometry>
-			</collision>
-		</link>
-		<joint name="${prefix}base2place_element_3">
-			<parent link="${prefix}base_link" />
-			<child link="${prefix}place_element_3" />
-			<origin xyz="0 0 0" rpy="0 0 0" />
-		</joint>
-		<link name="${prefix}pick_element_4">
-			<visual>
-				<geometry>
-					<mesh filename="package://assembly-instances/assembly_models/picknplace/bricks/meshes/collision/element_pick_4.stl" scale="0.001 0.001 0.001" />
-				</geometry>
-			</visual>
-			<collision>
-				<geometry>
-					<mesh filename="package://assembly-instances/assembly_models/picknplace/bricks/meshes/collision/element_pick_4.stl" scale="0.001 0.001 0.001" />
-				</geometry>
-			</collision>
-		</link>
-		<joint name="${prefix}base2pick_element_4">
-			<parent link="${prefix}base_link" />
-			<child link="${prefix}pick_element_4" />
-			<origin xyz="0 0 0" rpy="0 0 0" />
-		</joint>
-		<link name="${prefix}place_element_4">
-			<visual>
-				<geometry>
-					<mesh filename="package://assembly-instances/assembly_models/picknplace/bricks/meshes/collision/element_place_4.stl" scale="0.001 0.001 0.001" />
-				</geometry>
-			</visual>
-			<collision>
-				<geometry>
-					<mesh filename="package://assembly-instances/assembly_models/picknplace/bricks/meshes/collision/element_place_4.stl" scale="0.001 0.001 0.001" />
-				</geometry>
-			</collision>
-		</link>
-		<link name="${prefix}place_element_4">
-			<visual>
-				<geometry>
-					<mesh filename="package://assembly-instances/assembly_models/picknplace/bricks/meshes/collision/element_place_4.stl" scale="0.001 0.001 0.001" />
-				</geometry>
-			</visual>
-			<collision>
-				<geometry>
-					<mesh filename="package://assembly-instances/assembly_models/picknplace/bricks/meshes/collision/element_place_4.stl" scale="0.001 0.001 0.001" />
-				</geometry>
-			</collision>
-		</link>
-		<joint name="${prefix}base2place_element_4">
-			<parent link="${prefix}base_link" />
-			<child link="${prefix}place_element_4" />
-			<origin xyz="0 0 0" rpy="0 0 0" />
-		</joint>
-		<link name="${prefix}pick_element_5">
-			<visual>
-				<geometry>
-					<mesh filename="package://assembly-instances/assembly_models/picknplace/bricks/meshes/collision/element_pick_5.stl" scale="0.001 0.001 0.001" />
-				</geometry>
-			</visual>
-			<collision>
-				<geometry>
-					<mesh filename="package://assembly-instances/assembly_models/picknplace/bricks/meshes/collision/element_pick_5.stl" scale="0.001 0.001 0.001" />
-				</geometry>
-			</collision>
-		</link>
-		<joint name="${prefix}base2pick_element_5">
-			<parent link="${prefix}base_link" />
-			<child link="${prefix}pick_element_5" />
-			<origin xyz="0 0 0" rpy="0 0 0" />
-		</joint>
-		<link name="${prefix}place_element_5">
-			<visual>
-				<geometry>
-					<mesh filename="package://assembly-instances/assembly_models/picknplace/bricks/meshes/collision/element_place_5.stl" scale="0.001 0.001 0.001" />
-				</geometry>
-			</visual>
-			<collision>
-				<geometry>
-					<mesh filename="package://assembly-instances/assembly_models/picknplace/bricks/meshes/collision/element_place_5.stl" scale="0.001 0.001 0.001" />
-				</geometry>
-			</collision>
-		</link>
-		<link name="${prefix}place_element_5">
-			<visual>
-				<geometry>
-					<mesh filename="package://assembly-instances/assembly_models/picknplace/bricks/meshes/collision/element_place_5.stl" scale="0.001 0.001 0.001" />
-				</geometry>
-			</visual>
-			<collision>
-				<geometry>
-					<mesh filename="package://assembly-instances/assembly_models/picknplace/bricks/meshes/collision/element_place_5.stl" scale="0.001 0.001 0.001" />
-				</geometry>
-			</collision>
-		</link>
-		<joint name="${prefix}base2place_element_5">
-			<parent link="${prefix}base_link" />
-			<child link="${prefix}place_element_5" />
-			<origin xyz="0 0 0" rpy="0 0 0" />
-		</joint>
-		<link name="${prefix}pick_element_6">
-			<visual>
-				<geometry>
-					<mesh filename="package://assembly-instances/assembly_models/picknplace/bricks/meshes/collision/element_pick_6.stl" scale="0.001 0.001 0.001" />
-				</geometry>
-			</visual>
-			<collision>
-				<geometry>
-					<mesh filename="package://assembly-instances/assembly_models/picknplace/bricks/meshes/collision/element_pick_6.stl" scale="0.001 0.001 0.001" />
-				</geometry>
-			</collision>
-		</link>
-		<joint name="${prefix}base2pick_element_6">
-			<parent link="${prefix}base_link" />
-			<child link="${prefix}pick_element_6" />
-			<origin xyz="0 0 0" rpy="0 0 0" />
-		</joint>
-		<link name="${prefix}place_element_6">
-			<visual>
-				<geometry>
-					<mesh filename="package://assembly-instances/assembly_models/picknplace/bricks/meshes/collision/element_place_6.stl" scale="0.001 0.001 0.001" />
-				</geometry>
-			</visual>
-			<collision>
-				<geometry>
-					<mesh filename="package://assembly-instances/assembly_models/picknplace/bricks/meshes/collision/element_place_6.stl" scale="0.001 0.001 0.001" />
-				</geometry>
-			</collision>
-		</link>
-		<link name="${prefix}place_element_6">
-			<visual>
-				<geometry>
-					<mesh filename="package://assembly-instances/assembly_models/picknplace/bricks/meshes/collision/element_place_6.stl" scale="0.001 0.001 0.001" />
-				</geometry>
-			</visual>
-			<collision>
-				<geometry>
-					<mesh filename="package://assembly-instances/assembly_models/picknplace/bricks/meshes/collision/element_place_6.stl" scale="0.001 0.001 0.001" />
-				</geometry>
-			</collision>
-		</link>
-		<joint name="${prefix}base2place_element_6">
-			<parent link="${prefix}base_link" />
-			<child link="${prefix}place_element_6" />
-			<origin xyz="0 0 0" rpy="0 0 0" />
-		</joint>
-		<link name="${prefix}pick_element_7">
-			<visual>
-				<geometry>
-					<mesh filename="package://assembly-instances/assembly_models/picknplace/bricks/meshes/collision/element_pick_7.stl" scale="0.001 0.001 0.001" />
-				</geometry>
-			</visual>
-			<collision>
-				<geometry>
-					<mesh filename="package://assembly-instances/assembly_models/picknplace/bricks/meshes/collision/element_pick_7.stl" scale="0.001 0.001 0.001" />
-				</geometry>
-			</collision>
-		</link>
-		<joint name="${prefix}base2pick_element_7">
-			<parent link="${prefix}base_link" />
-			<child link="${prefix}pick_element_7" />
-			<origin xyz="0 0 0" rpy="0 0 0" />
-		</joint>
-		<link name="${prefix}place_element_7">
-			<visual>
-				<geometry>
-					<mesh filename="package://assembly-instances/assembly_models/picknplace/bricks/meshes/collision/element_place_7.stl" scale="0.001 0.001 0.001" />
-				</geometry>
-			</visual>
-			<collision>
-				<geometry>
-					<mesh filename="package://assembly-instances/assembly_models/picknplace/bricks/meshes/collision/element_place_7.stl" scale="0.001 0.001 0.001" />
-				</geometry>
-			</collision>
-		</link>
-		<link name="${prefix}place_element_7">
-			<visual>
-				<geometry>
-					<mesh filename="package://assembly-instances/assembly_models/picknplace/bricks/meshes/collision/element_place_7.stl" scale="0.001 0.001 0.001" />
-				</geometry>
-			</visual>
-			<collision>
-				<geometry>
-					<mesh filename="package://assembly-instances/assembly_models/picknplace/bricks/meshes/collision/element_place_7.stl" scale="0.001 0.001 0.001" />
-				</geometry>
-			</collision>
-		</link>
-		<joint name="${prefix}base2place_element_7">
-			<parent link="${prefix}base_link" />
-			<child link="${prefix}place_element_7" />
-			<origin xyz="0 0 0" rpy="0 0 0" />
-		</joint>
-		<link name="${prefix}pick_element_8">
-			<visual>
-				<geometry>
-					<mesh filename="package://assembly-instances/assembly_models/picknplace/bricks/meshes/collision/element_pick_8.stl" scale="0.001 0.001 0.001" />
-				</geometry>
-			</visual>
-			<collision>
-				<geometry>
-					<mesh filename="package://assembly-instances/assembly_models/picknplace/bricks/meshes/collision/element_pick_8.stl" scale="0.001 0.001 0.001" />
-				</geometry>
-			</collision>
-		</link>
-		<joint name="${prefix}base2pick_element_8">
-			<parent link="${prefix}base_link" />
-			<child link="${prefix}pick_element_8" />
-			<origin xyz="0 0 0" rpy="0 0 0" />
-		</joint>
-		<link name="${prefix}place_element_8">
-			<visual>
-				<geometry>
-					<mesh filename="package://assembly-instances/assembly_models/picknplace/bricks/meshes/collision/element_place_8.stl" scale="0.001 0.001 0.001" />
-				</geometry>
-			</visual>
-			<collision>
-				<geometry>
-					<mesh filename="package://assembly-instances/assembly_models/picknplace/bricks/meshes/collision/element_place_8.stl" scale="0.001 0.001 0.001" />
-				</geometry>
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