Commit message: add obj files for the picknplace instance. Accompanied json file chaned accordingly.

File: assembly_models/picknplace/bricks/urdf/brick_demo.xacro (robot description, xacro)
@@ -1,10 +1,10 @@
-﻿<?xml version="1.0" ?>
+﻿<?xml version="1.0" encoding="utf-8"?>
 <robot name="brick_demo" xmlns:xacro="http://wiki.ros.org/xacro">
 	<xacro:include filename="$(find assembly-instances)/assembly_models/picknplace/bricks/urdf/brick_demo_geometry.xacro" />
-	<xacro:brick_demo_geometry prefix="ws_" />
+	<xacro:brick_demo_geometry prefix="workspace_geo_" />
 	<link name="base_link" />
 	<joint name="world2workspace_geo" type="fixed">
 		<parent link="base_link" />
-		<child link="ws_base_link" />
+		<child link="workspace_geo_base_link" />
 		<origin xyz="0 0 0" rpy="0 0 0" />
 	</joint>

File: assembly_models/picknplace/bricks/urdf/brick_demo_geometry.xacro (robot description, xacro)
@@ -1,3 +1,3 @@
-﻿<?xml version="1.0" ?>
+﻿<?xml version="1.0" encoding="utf-8"?>
 <robot xmlns:xacro="http://wiki.ros.org/xacro">
 	<xacro:macro name="brick_demo_geometry" params="prefix">
@@ -6,10 +6,10 @@
 			<visual>
 				<geometry>
-					<mesh filename="$(find assembly-instances)/assembly_models/picknplace/bricks/meshes/collision/element_pick_0.stl" scale="0.001 0.001 0.001" />
-				</geometry>
-			</visual>
-			<collision>
-				<geometry>
-					<mesh filename="$(find assembly-instances)/assembly_models/picknplace/bricks/meshes/collision/element_pick_0.stl" scale="0.001 0.001 0.001" />
+					<mesh filename="$(find assembly-instances)/assembly_models/picknplace/bricks/meshes/collision/element_pick_0.obj" scale="0.001 0.001 0.001" />
+				</geometry>
+			</visual>
+			<collision>
+				<geometry>
+					<mesh filename="$(find assembly-instances)/assembly_models/picknplace/bricks/meshes/collision/element_pick_0.obj" scale="0.001 0.001 0.001" />
 				</geometry>
 			</collision>
@@ -23,10 +23,10 @@
 			<visual>
 				<geometry>
-					<mesh filename="$(find assembly-instances)/assembly_models/picknplace/bricks/meshes/collision/element_place_0.stl" scale="0.001 0.001 0.001" />
-				</geometry>
-			</visual>
-			<collision>
-				<geometry>
-					<mesh filename="$(find assembly-instances)/assembly_models/picknplace/bricks/meshes/collision/element_place_0.stl" scale="0.001 0.001 0.001" />
+					<mesh filename="$(find assembly-instances)/assembly_models/picknplace/bricks/meshes/collision/element_place_0.obj" scale="0.001 0.001 0.001" />
+				</geometry>
+			</visual>
+			<collision>
+				<geometry>
+					<mesh filename="$(find assembly-instances)/assembly_models/picknplace/bricks/meshes/collision/element_place_0.obj" scale="0.001 0.001 0.001" />
 				</geometry>
 			</collision>
@@ -40,10 +40,10 @@
 			<visual>
 				<geometry>
-					<mesh filename="$(find assembly-instances)/assembly_models/picknplace/bricks/meshes/collision/element_pick_1.stl" scale="0.001 0.001 0.001" />
-				</geometry>
-			</visual>
-			<collision>
-				<geometry>
-					<mesh filename="$(find assembly-instances)/assembly_models/picknplace/bricks/meshes/collision/element_pick_1.stl" scale="0.001 0.001 0.001" />
+					<mesh filename="$(find assembly-instances)/assembly_models/picknplace/bricks/meshes/collision/element_pick_1.obj" scale="0.001 0.001 0.001" />
+				</geometry>
+			</visual>
+			<collision>
+				<geometry>
+					<mesh filename="$(find assembly-instances)/assembly_models/picknplace/bricks/meshes/collision/element_pick_1.obj" scale="0.001 0.001 0.001" />
 				</geometry>
 			</collision>
@@ -57,10 +57,10 @@
 			<visual>
 				<geometry>
-					<mesh filename="$(find assembly-instances)/assembly_models/picknplace/bricks/meshes/collision/element_place_1.stl" scale="0.001 0.001 0.001" />
-				</geometry>
-			</visual>
-			<collision>
-				<geometry>
-					<mesh filename="$(find assembly-instances)/assembly_models/picknplace/bricks/meshes/collision/element_place_1.stl" scale="0.001 0.001 0.001" />
+					<mesh filename="$(find assembly-instances)/assembly_models/picknplace/bricks/meshes/collision/element_place_1.obj" scale="0.001 0.001 0.001" />
+				</geometry>
+			</visual>
+			<collision>
+				<geometry>
+					<mesh filename="$(find assembly-instances)/assembly_models/picknplace/bricks/meshes/collision/element_place_1.obj" scale="0.001 0.001 0.001" />
 				</geometry>
 			</collision>
@@ -74,10 +74,10 @@
 			<visual>
 				<geometry>
-					<mesh filename="$(find assembly-instances)/assembly_models/picknplace/bricks/meshes/collision/element_pick_2.stl" scale="0.001 0.001 0.001" />
-				</geometry>
-			</visual>
-			<collision>
-				<geometry>
-					<mesh filename="$(find assembly-instances)/assembly_models/picknplace/bricks/meshes/collision/element_pick_2.stl" scale="0.001 0.001 0.001" />
+					<mesh filename="$(find assembly-instances)/assembly_models/picknplace/bricks/meshes/collision/element_pick_2.obj" scale="0.001 0.001 0.001" />
+				</geometry>
+			</visual>
+			<collision>
+				<geometry>
+					<mesh filename="$(find assembly-instances)/assembly_models/picknplace/bricks/meshes/collision/element_pick_2.obj" scale="0.001 0.001 0.001" />
 				</geometry>
 			</collision>
@@ -91,10 +91,10 @@
 			<visual>
 				<geometry>
-					<mesh filename="$(find assembly-instances)/assembly_models/picknplace/bricks/meshes/collision/element_place_2.stl" scale="0.001 0.001 0.001" />
-				</geometry>
-			</visual>
-			<collision>
-				<geometry>
-					<mesh filename="$(find assembly-instances)/assembly_models/picknplace/bricks/meshes/collision/element_place_2.stl" scale="0.001 0.001 0.001" />
+					<mesh filename="$(find assembly-instances)/assembly_models/picknplace/bricks/meshes/collision/element_place_2.obj" scale="0.001 0.001 0.001" />
+				</geometry>
+			</visual>
+			<collision>
+				<geometry>
+					<mesh filename="$(find assembly-instances)/assembly_models/picknplace/bricks/meshes/collision/element_place_2.obj" scale="0.001 0.001 0.001" />
 				</geometry>
 			</collision>
@@ -108,10 +108,10 @@
 			<visual>
 				<geometry>
-					<mesh filename="$(find assembly-instances)/assembly_models/picknplace/bricks/meshes/collision/element_pick_3.stl" scale="0.001 0.001 0.001" />
-				</geometry>
-			</visual>
-			<collision>
-				<geometry>
-					<mesh filename="$(find assembly-instances)/assembly_models/picknplace/bricks/meshes/collision/element_pick_3.stl" scale="0.001 0.001 0.001" />
+					<mesh filename="$(find assembly-instances)/assembly_models/picknplace/bricks/meshes/collision/element_pick_3.obj" scale="0.001 0.001 0.001" />
+				</geometry>
+			</visual>
+			<collision>
+				<geometry>
+					<mesh filename="$(find assembly-instances)/assembly_models/picknplace/bricks/meshes/collision/element_pick_3.obj" scale="0.001 0.001 0.001" />
 				</geometry>
 			</collision>
@@ -125,10 +125,10 @@
 			<visual>
 				<geometry>
-					<mesh filename="$(find assembly-instances)/assembly_models/picknplace/bricks/meshes/collision/element_place_3.stl" scale="0.001 0.001 0.001" />
-				</geometry>
-			</visual>
-			<collision>
-				<geometry>
-					<mesh filename="$(find assembly-instances)/assembly_models/picknplace/bricks/meshes/collision/element_place_3.stl" scale="0.001 0.001 0.001" />
+					<mesh filename="$(find assembly-instances)/assembly_models/picknplace/bricks/meshes/collision/element_place_3.obj" scale="0.001 0.001 0.001" />
+				</geometry>
+			</visual>
+			<collision>
+				<geometry>
+					<mesh filename="$(find assembly-instances)/assembly_models/picknplace/bricks/meshes/collision/element_place_3.obj" scale="0.001 0.001 0.001" />
 				</geometry>
 			</collision>
@@ -142,10 +142,10 @@
 			<visual>
 				<geometry>
-					<mesh filename="$(find assembly-instances)/assembly_models/picknplace/bricks/meshes/collision/element_pick_4.stl" scale="0.001 0.001 0.001" />
-				</geometry>
-			</visual>
-			<collision>
-				<geometry>
-					<mesh filename="$(find assembly-instances)/assembly_models/picknplace/bricks/meshes/collision/element_pick_4.stl" scale="0.001 0.001 0.001" />
+					<mesh filename="$(find assembly-instances)/assembly_models/picknplace/bricks/meshes/collision/element_pick_4.obj" scale="0.001 0.001 0.001" />
+				</geometry>
+			</visual>
+			<collision>
+				<geometry>
+					<mesh filename="$(find assembly-instances)/assembly_models/picknplace/bricks/meshes/collision/element_pick_4.obj" scale="0.001 0.001 0.001" />
 				</geometry>
 			</collision>
@@ -159,10 +159,10 @@
 			<visual>
 				<geometry>
-					<mesh filename="$(find assembly-instances)/assembly_models/picknplace/bricks/meshes/collision/element_place_4.stl" scale="0.001 0.001 0.001" />
-				</geometry>
-			</visual>
-			<collision>
-				<geometry>
-					<mesh filename="$(find assembly-instances)/assembly_models/picknplace/bricks/meshes/collision/element_place_4.stl" scale="0.001 0.001 0.001" />
+					<mesh filename="$(find assembly-instances)/assembly_models/picknplace/bricks/meshes/collision/element_place_4.obj" scale="0.001 0.001 0.001" />
+				</geometry>
+			</visual>
+			<collision>
+				<geometry>
+					<mesh filename="$(find assembly-instances)/assembly_models/picknplace/bricks/meshes/collision/element_place_4.obj" scale="0.001 0.001 0.001" />
 				</geometry>
 			</collision>
@@ -176,10 +176,10 @@
 			<visual>
 				<geometry>
-					<mesh filename="$(find assembly-instances)/assembly_models/picknplace/bricks/meshes/collision/element_pick_5.stl" scale="0.001 0.001 0.001" />
-				</geometry>
-			</visual>
-			<collision>
-				<geometry>
-					<mesh filename="$(find assembly-instances)/assembly_models/picknplace/bricks/meshes/collision/element_pick_5.stl" scale="0.001 0.001 0.001" />
+					<mesh filename="$(find assembly-instances)/assembly_models/picknplace/bricks/meshes/collision/element_pick_5.obj" scale="0.001 0.001 0.001" />
+				</geometry>
+			</visual>
+			<collision>
+				<geometry>
+					<mesh filename="$(find assembly-instances)/assembly_models/picknplace/bricks/meshes/collision/element_pick_5.obj" scale="0.001 0.001 0.001" />
 				</geometry>
 			</collision>
@@ -193,10 +193,10 @@
 			<visual>
 				<geometry>
-					<mesh filename="$(find assembly-instances)/assembly_models/picknplace/bricks/meshes/collision/element_place_5.stl" scale="0.001 0.001 0.001" />
-				</geometry>
-			</visual>
-			<collision>
-				<geometry>
-					<mesh filename="$(find assembly-instances)/assembly_models/picknplace/bricks/meshes/collision/element_place_5.stl" scale="0.001 0.001 0.001" />
+					<mesh filename="$(find assembly-instances)/assembly_models/picknplace/bricks/meshes/collision/element_place_5.obj" scale="0.001 0.001 0.001" />
+				</geometry>
+			</visual>
+			<collision>
+				<geometry>
+					<mesh filename="$(find assembly-instances)/assembly_models/picknplace/bricks/meshes/collision/element_place_5.obj" scale="0.001 0.001 0.001" />
 				</geometry>
 			</collision>
@@ -210,10 +210,10 @@
 			<visual>
 				<geometry>
-					<mesh filename="$(find assembly-instances)/assembly_models/picknplace/bricks/meshes/collision/element_pick_6.stl" scale="0.001 0.001 0.001" />
-				</geometry>
-			</visual>
-			<collision>
-				<geometry>
-					<mesh filename="$(find assembly-instances)/assembly_models/picknplace/bricks/meshes/collision/element_pick_6.stl" scale="0.001 0.001 0.001" />
+					<mesh filename="$(find assembly-instances)/assembly_models/picknplace/bricks/meshes/collision/element_pick_6.obj" scale="0.001 0.001 0.001" />
+				</geometry>
+			</visual>
+			<collision>
+				<geometry>
+					<mesh filename="$(find assembly-instances)/assembly_models/picknplace/bricks/meshes/collision/element_pick_6.obj" scale="0.001 0.001 0.001" />
 				</geometry>
 			</collision>
@@ -227,10 +227,10 @@
 			<visual>
 				<geometry>
-					<mesh filename="$(find assembly-instances)/assembly_models/picknplace/bricks/meshes/collision/element_place_6.stl" scale="0.001 0.001 0.001" />
-				</geometry>
-			</visual>
-			<collision>
-				<geometry>
-					<mesh filename="$(find assembly-instances)/assembly_models/picknplace/bricks/meshes/collision/element_place_6.stl" scale="0.001 0.001 0.001" />
+					<mesh filename="$(find assembly-instances)/assembly_models/picknplace/bricks/meshes/collision/element_place_6.obj" scale="0.001 0.001 0.001" />
+				</geometry>
+			</visual>
+			<collision>
+				<geometry>
+					<mesh filename="$(find assembly-instances)/assembly_models/picknplace/bricks/meshes/collision/element_place_6.obj" scale="0.001 0.001 0.001" />
 				</geometry>
 			</collision>
@@ -244,10 +244,10 @@
 			<visual>
 				<geometry>
-					<mesh filename="$(find assembly-instances)/assembly_models/picknplace/bricks/meshes/collision/element_pick_7.stl" scale="0.001 0.001 0.001" />
-				</geometry>
-			</visual>
-			<collision>
-				<geometry>
-					<mesh filename="$(find assembly-instances)/assembly_models/picknplace/bricks/meshes/collision/element_pick_7.stl" scale="0.001 0.001 0.001" />
+					<mesh filename="$(find assembly-instances)/assembly_models/picknplace/bricks/meshes/collision/element_pick_7.obj" scale="0.001 0.001 0.001" />
+				</geometry>
+			</visual>
+			<collision>
+				<geometry>
+					<mesh filename="$(find assembly-instances)/assembly_models/picknplace/bricks/meshes/collision/element_pick_7.obj" scale="0.001 0.001 0.001" />
 				</geometry>
 			</collision>
@@ -261,10 +261,10 @@
 			<visual>
 				<geometry>
-					<mesh filename="$(find assembly-instances)/assembly_models/picknplace/bricks/meshes/collision/element_place_7.stl" scale="0.001 0.001 0.001" />
-				</geometry>
-			</visual>
-			<collision>
-				<geometry>
-					<mesh filename="$(find assembly-instances)/assembly_models/picknplace/bricks/meshes/collision/element_place_7.stl" scale="0.001 0.001 0.001" />
+					<mesh filename="$(find assembly-instances)/assembly_models/picknplace/bricks/meshes/collision/element_place_7.obj" scale="0.001 0.001 0.001" />
+				</geometry>
+			</visual>
+			<collision>
+				<geometry>
+					<mesh filename="$(find assembly-instances)/assembly_models/picknplace/bricks/meshes/collision/element_place_7.obj" scale="0.001 0.001 0.001" />
 				</geometry>
 			</collision>
@@ -278,10 +278,10 @@
 			<visual>
 				<geometry>
-					<mesh filename="$(find assembly-instances)/assembly_models/picknplace/bricks/meshes/collision/element_pick_8.stl" scale="0.001 0.001 0.001" />
-				</geometry>
-			</visual>
-			<collision>
-				<geometry>
-					<mesh filename="$(find assembly-instances)/assembly_models/picknplace/bricks/meshes/collision/element_pick_8.stl" scale="0.001 0.001 0.001" />
+					<mesh filename="$(find assembly-instances)/assembly_models/picknplace/bricks/meshes/collision/element_pick_8.obj" scale="0.001 0.001 0.001" />
+				</geometry>
+			</visual>
+			<collision>
+				<geometry>
+					<mesh filename="$(find assembly-instances)/assembly_models/picknplace/bricks/meshes/collision/element_pick_8.obj" scale="0.001 0.001 0.001" />
 				</geometry>
 			</collision>
@@ -295,10 +295,10 @@
 			<visual>
 				<geometry>
-					<mesh filename="$(find assembly-instances)/assembly_models/picknplace/bricks/meshes/collision/element_place_8.stl" scale="0.001 0.001 0.001" />
-				</geometry>
-			</visual>
-			<collision>
-				<geometry>
-					<mesh filename="$(find assembly-instances)/assembly_models/picknplace/bricks/meshes/collision/element_place_8.stl" scale="0.001 0.001 0.001" />
+					<mesh filename="$(find assembly-instances)/assembly_models/picknplace/bricks/meshes/collision/element_place_8.obj" scale="0.001 0.001 0.001" />
+				</geometry>
+			</visual>
+			<collision>
+				<geometry>
+					<mesh filename="$(find assembly-instances)/assembly_models/picknplace/bricks/meshes/collision/element_place_8.obj" scale="0.001 0.001 0.001" />
 				</geometry>
 			</collision>
@@ -312,10 +312,10 @@
 			<visual>
 				<geometry>
-					<mesh filename="$(find assembly-instances)/assembly_models/picknplace/bricks/meshes/collision/element_pick_9.stl" scale="0.001 0.001 0.001" />
-				</geometry>
-			</visual>
-			<collision>
-				<geometry>
-					<mesh filename="$(find assembly-instances)/assembly_models/picknplace/bricks/meshes/collision/element_pick_9.stl" scale="0.001 0.001 0.001" />
+					<mesh filename="$(find assembly-instances)/assembly_models/picknplace/bricks/meshes/collision/element_pick_9.obj" scale="0.001 0.001 0.001" />
+				</geometry>
+			</visual>
+			<collision>
+				<geometry>
+					<mesh filename="$(find assembly-instances)/assembly_models/picknplace/bricks/meshes/collision/element_pick_9.obj" scale="0.001 0.001 0.001" />
 				</geometry>
 			</collision>
@@ -329,10 +329,10 @@
 			<visual>
 				<geometry>
-					<mesh filename="$(find assembly-instances)/assembly_models/picknplace/bricks/meshes/collision/element_place_9.stl" scale="0.001 0.001 0.001" />
-				</geometry>
-			</visual>
-			<collision>
-				<geometry>
-					<mesh filename="$(find assembly-instances)/assembly_models/picknplace/bricks/meshes/collision/element_place_9.stl" scale="0.001 0.001 0.001" />
+					<mesh filename="$(find assembly-instances)/assembly_models/picknplace/bricks/meshes/collision/element_place_9.obj" scale="0.001 0.001 0.001" />
+				</geometry>
+			</visual>
+			<collision>
+				<geometry>
+					<mesh filename="$(find assembly-instances)/assembly_models/picknplace/bricks/meshes/collision/element_place_9.obj" scale="0.001 0.001 0.001" />
 				</geometry>
 			</collision>
@@ -346,10 +346,10 @@
 			<visual>
 				<geometry>
-					<mesh filename="$(find assembly-instances)/assembly_models/picknplace/bricks/meshes/collision/element_pick_10.stl" scale="0.001 0.001 0.001" />
-				</geometry>
-			</visual>
-			<collision>
-				<geometry>
-					<mesh filename="$(find assembly-instances)/assembly_models/picknplace/bricks/meshes/collision/element_pick_10.stl" scale="0.001 0.001 0.001" />
+					<mesh filename="$(find assembly-instances)/assembly_models/picknplace/bricks/meshes/collision/element_pick_10.obj" scale="0.001 0.001 0.001" />
+				</geometry>
+			</visual>
+			<collision>
+				<geometry>
+					<mesh filename="$(find assembly-instances)/assembly_models/picknplace/bricks/meshes/collision/element_pick_10.obj" scale="0.001 0.001 0.001" />
 				</geometry>
 			</collision>
@@ -363,10 +363,10 @@
 			<visual>
 				<geometry>
-					<mesh filename="$(find assembly-instances)/assembly_models/picknplace/bricks/meshes/collision/element_place_10.stl" scale="0.001 0.001 0.001" />
-				</geometry>
-			</visual>
-			<collision>
-				<geometry>
-					<mesh filename="$(find assembly-instances)/assembly_models/picknplace/bricks/meshes/collision/element_place_10.stl" scale="0.001 0.001 0.001" />
+					<mesh filename="$(find assembly-instances)/assembly_models/picknplace/bricks/meshes/collision/element_place_10.obj" scale="0.001 0.001 0.001" />
+				</geometry>
+			</visual>
+			<collision>
+				<geometry>
+					<mesh filename="$(find assembly-instances)/assembly_models/picknplace/bricks/meshes/collision/element_place_10.obj" scale="0.001 0.001 0.001" />
 				</geometry>
 			</collision>
@@ -380,10 +380,10 @@
 			<visual>
 				<geometry>
-					<mesh filename="$(find assembly-instances)/assembly_models/picknplace/bricks/meshes/collision/element_pick_11.stl" scale="0.001 0.001 0.001" />
-				</geometry>
-			</visual>
-			<collision>
-				<geometry>
-					<mesh filename="$(find assembly-instances)/assembly_models/picknplace/bricks/meshes/collision/element_pick_11.stl" scale="0.001 0.001 0.001" />
+					<mesh filename="$(find assembly-instances)/assembly_models/picknplace/bricks/meshes/collision/element_pick_11.obj" scale="0.001 0.001 0.001" />
+				</geometry>
+			</visual>
+			<collision>
+				<geometry>
+					<mesh filename="$(find assembly-instances)/assembly_models/picknplace/bricks/meshes/collision/element_pick_11.obj" scale="0.001 0.001 0.001" />
 				</geometry>
 			</collision>
@@ -397,10 +397,10 @@
 			<visual>
 				<geometry>
-					<mesh filename="$(find assembly-instances)/assembly_models/picknplace/bricks/meshes/collision/element_place_11.stl" scale="0.001 0.001 0.001" />
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