Commit message: swap in files that are used by pb-construction.

File: picknplace/bricks/urdf/brick_demo.urdf (robot description, URDF)
Before this commit: robot brick_demo, 39 links, 38 joints
Links:
- link workspace_geo_pick_element_0: geometry collision mesh filename=../meshes/collision/element_pick_0.obj scale=0.001 0.001 0.001; visual mesh filename=../meshes/collision/element_pick_0.obj scale=0.001 0.001 0.001
- link workspace_geo_pick_element_1: geometry collision mesh filename=../meshes/collision/element_pick_1.obj scale=0.001 0.001 0.001; visual mesh filename=../meshes/collision/element_pick_1.obj scale=0.001 0.001 0.001
- link workspace_geo_pick_element_10: geometry collision mesh filename=../meshes/collision/element_pick_10.obj scale=0.001 0.001 0.001; visual mesh filename=../meshes/collision/element_pick_10.obj scale=0.001 0.001 0.001
- link workspace_geo_pick_element_11: geometry collision mesh filename=../meshes/collision/element_pick_11.obj scale=0.001 0.001 0.001; visual mesh filename=../meshes/collision/element_pick_11.obj scale=0.001 0.001 0.001
- link workspace_geo_pick_element_2: geometry collision mesh filename=../meshes/collision/element_pick_2.obj scale=0.001 0.001 0.001; visual mesh filename=../meshes/collision/element_pick_2.obj scale=0.001 0.001 0.001
- link workspace_geo_pick_element_3: geometry collision mesh filename=../meshes/collision/element_pick_3.obj scale=0.001 0.001 0.001; visual mesh filename=../meshes/collision/element_pick_3.obj scale=0.001 0.001 0.001
- link workspace_geo_pick_element_4: geometry collision mesh filename=../meshes/collision/element_pick_4.obj scale=0.001 0.001 0.001; visual mesh filename=../meshes/collision/element_pick_4.obj scale=0.001 0.001 0.001
- link workspace_geo_pick_element_5: geometry collision mesh filename=../meshes/collision/element_pick_5.obj scale=0.001 0.001 0.001; visual mesh filename=../meshes/collision/element_pick_5.obj scale=0.001 0.001 0.001
- link workspace_geo_pick_element_6: geometry collision mesh filename=../meshes/collision/element_pick_6.obj scale=0.001 0.001 0.001; visual mesh filename=../meshes/collision/element_pick_6.obj scale=0.001 0.001 0.001
- link workspace_geo_pick_element_7: geometry collision mesh filename=../meshes/collision/element_pick_7.obj scale=0.001 0.001 0.001; visual mesh filename=../meshes/collision/element_pick_7.obj scale=0.001 0.001 0.001
- link workspace_geo_pick_element_8: geometry collision mesh filename=../meshes/collision/element_pick_8.obj scale=0.001 0.001 0.001; visual mesh filename=../meshes/collision/element_pick_8.obj scale=0.001 0.001 0.001
- link workspace_geo_pick_element_9: geometry collision mesh filename=../meshes/collision/element_pick_9.obj scale=0.001 0.001 0.001; visual mesh filename=../meshes/collision/element_pick_9.obj scale=0.001 0.001 0.001
- link workspace_geo_pick_support_object_0: geometry collision mesh filename=../meshes/collision/support_place_table.obj scale=0.001 0.001 0.001; visual mesh filename=../meshes/collision/support_place_table.obj scale=0.001 0.001 0.001
- link workspace_geo_place_element_0: geometry collision mesh filename=../meshes/collision/element_place_0.obj scale=0.001 0.001 0.001; visual mesh filename=../meshes/collision/element_place_0.obj scale=0.001 0.001 0.001
- link workspace_geo_place_element_1: geometry collision mesh filename=../meshes/collision/element_place_1.obj scale=0.001 0.001 0.001; visual mesh filename=../meshes/collision/element_place_1.obj scale=0.001 0.001 0.001
- link workspace_geo_place_element_10: geometry collision mesh filename=../meshes/collision/element_place_10.obj scale=0.001 0.001 0.001; visual mesh filename=../meshes/collision/element_place_10.obj scale=0.001 0.001 0.001
- link workspace_geo_place_element_11: geometry collision mesh filename=../meshes/collision/element_place_11.obj scale=0.001 0.001 0.001; visual mesh filename=../meshes/collision/element_place_11.obj scale=0.001 0.001 0.001
- link workspace_geo_place_element_2: geometry collision mesh filename=../meshes/collision/element_place_2.obj scale=0.001 0.001 0.001; visual mesh filename=../meshes/collision/element_place_2.obj scale=0.001 0.001 0.001
- link workspace_geo_place_element_3: geometry collision mesh filename=../meshes/collision/element_place_3.obj scale=0.001 0.001 0.001; visual mesh filename=../meshes/collision/element_place_3.obj scale=0.001 0.001 0.001
- link workspace_geo_place_element_4: geometry collision mesh filename=../meshes/collision/element_place_4.obj scale=0.001 0.001 0.001; visual mesh filename=../meshes/collision/element_place_4.obj scale=0.001 0.001 0.001
- link workspace_geo_place_element_5: geometry collision mesh filename=../meshes/collision/element_place_5.obj scale=0.001 0.001 0.001; visual mesh filename=../meshes/collision/element_place_5.obj scale=0.001 0.001 0.001
- link workspace_geo_place_element_6: geometry collision mesh filename=../meshes/collision/element_place_6.obj scale=0.001 0.001 0.001; visual mesh filename=../meshes/collision/element_place_6.obj scale=0.001 0.001 0.001
- link workspace_geo_place_element_7: geometry collision mesh filename=../meshes/collision/element_place_7.obj scale=0.001 0.001 0.001; visual mesh filename=../meshes/collision/element_place_7.obj scale=0.001 0.001 0.001
- link workspace_geo_place_element_8: geometry collision mesh filename=../meshes/collision/element_place_8.obj scale=0.001 0.001 0.001; visual mesh filename=../meshes/collision/element_place_8.obj scale=0.001 0.001 0.001
- link workspace_geo_place_element_9: geometry collision mesh filename=../meshes/collision/element_place_9.obj scale=0.001 0.001 0.001; visual mesh filename=../meshes/collision/element_place_9.obj scale=0.001 0.001 0.001
- link workspace_geo_place_support_object_0: geometry collision mesh filename=../meshes/collision/pick_left_over_bricks_0.obj scale=0.001 0.001 0.001; visual mesh filename=../meshes/collision/pick_left_over_bricks_0.obj scale=0.001 0.001 0.001
- link workspace_geo_place_support_object_1: geometry collision mesh filename=../meshes/collision/pick_left_over_bricks_1.obj scale=0.001 0.001 0.001; visual mesh filename=../meshes/collision/pick_left_over_bricks_1.obj scale=0.001 0.001 0.001
- link workspace_geo_place_support_object_10: geometry collision mesh filename=../meshes/collision/pick_left_over_bricks_10.obj scale=0.001 0.001 0.001; visual mesh filename=../meshes/collision/pick_left_over_bricks_10.obj scale=0.001 0.001 0.001
- link workspace_geo_place_support_object_11: geometry collision mesh filename=../meshes/collision/pick_left_over_bricks_11.obj scale=0.001 0.001 0.001; visual mesh filename=../meshes/collision/pick_left_over_bricks_11.obj scale=0.001 0.001 0.001
- link workspace_geo_place_support_object_2: geometry collision mesh filename=../meshes/collision/pick_left_over_bricks_4.obj scale=0.001 0.001 0.001; visual mesh filename=../meshes/collision/pick_left_over_bricks_4.obj scale=0.001 0.001 0.001
- link workspace_geo_place_support_object_3: geometry collision mesh filename=../meshes/collision/pick_left_over_bricks_2.obj scale=0.001 0.001 0.001; visual mesh filename=../meshes/collision/pick_left_over_bricks_2.obj scale=0.001 0.001 0.001
- link workspace_geo_place_support_object_4: geometry collision mesh filename=../meshes/collision/pick_left_over_bricks_5.obj scale=0.001 0.001 0.001; visual mesh filename=../meshes/collision/pick_left_over_bricks_5.obj scale=0.001 0.001 0.001
- link workspace_geo_place_support_object_5: geometry collision mesh filename=../meshes/collision/pick_left_over_bricks_3.obj scale=0.001 0.001 0.001; visual mesh filename=../meshes/collision/pick_left_over_bricks_3.obj scale=0.001 0.001 0.001
- link workspace_geo_place_support_object_6: geometry collision mesh filename=../meshes/collision/pick_left_over_bricks_6.obj scale=0.001 0.001 0.001; visual mesh filename=../meshes/collision/pick_left_over_bricks_6.obj scale=0.001 0.001 0.001
- link workspace_geo_place_support_object_7: geometry collision mesh filename=../meshes/collision/pick_left_over_bricks_7.obj scale=0.001 0.001 0.001; visual mesh filename=../meshes/collision/pick_left_over_bricks_7.obj scale=0.001 0.001 0.001
- link workspace_geo_place_support_object_8: geometry collision mesh filename=../meshes/collision/pick_left_over_bricks_8.obj scale=0.001 0.001 0.001; visual mesh filename=../meshes/collision/pick_left_over_bricks_8.obj scale=0.001 0.001 0.001
- link workspace_geo_place_support_object_9: geometry collision mesh filename=../meshes/collision/pick_left_over_bricks_9.obj scale=0.001 0.001 0.001; visual mesh filename=../meshes/collision/pick_left_over_bricks_9.obj scale=0.001 0.001 0.001
